File: kb/_autosave-kb.kicad_pcb (KiCad board)
At the start: 2 copper layers, 108 parts, among them J1 Conn_01x04_MountingPin, SW1 SW_Push, SW10 SW_Push, SW11 SW_Push, SW12 SW_Push, SW13 SW_Push, SW14 SW_Push, SW15 SW_Push, SW16 SW_Push, SW17 SW_Push, SW18 SW_Push, SW19 SW_Push, SW2 SW_Push, SW20 SW_Push, SW21 SW_Push, SW22 SW_Push, SW23 SW_Push, SW24 SW_Push, SW25 SW_Push, SW26 SW_Push, SW27 SW_Push, SW28 SW_Push, SW29 SW_Push, SW3 SW_Push, SW30 SW_Push, SW31 SW_Push, SW32 SW_Push, SW33 SW_Push, SW34 SW_Push, SW35 SW_Push, SW36 SW_Push, SW37 SW_Push, SW38 SW_Push, SW39 SW_Push, SW4 SW_Push, SW40 SW_Push, SW41 SW_Push, SW42 SW_Push, SW43 SW_Push, SW44 SW_Push, SW45 SW_Push, SW46 SW_Push, SW48 SW_Push, SW5 SW_Push, SW6 SW_Push, SW7 SW_Push, SW8 SW_Push, SW9 SW_Push, U2 STM32G474CETx, U4 XC6206PxxxMR

Commit message: Added NSRT, Fixed Pins
Fixed boot pin and reset pin assignments, rerouted accordingly
Parts:
- added C6: 100nF, Capacitor_SMD:C_0805_2012Metric, B.Cu at (200.8, 86.9)
- added SW47: RESET, Button_Switch_SMD:SW_SPST_SKQG_WithStem, B.Cu at (271.4, 33.9)
- SW48: value SW_Push -> BOOT
- moved R5 59.3 mm to (241.9, 32.0), turned to -90 degrees
- moved SW48 25.0 mm to (247.4, 34.3)
- moved D42 8.87 mm to (181.0, 93.6)
- moved C1 1.04 mm to (202.7, 98.9), turned to 45 degrees
- moved C3 1.02 mm to (197.2, 85.5), turned to 45 degrees
- moved C5 1.02 mm to (187.5, 93.2), turned to -135 degrees
- moved C4 0.13 mm to (202.4, 102.4)
Connections:
- U2 pad 13: ROW3 -> ROW2
- U2 pad 31: unconnected-(U2-PA9-Pad31) -> ROW3
- U2 pad 44: ROW0 -> COL7
- U2 pad 45: ROW1 -> BOOT
- U2 pad 46: ROW2 -> ROW1
- U2 pad 7: BOOT -> RESET
- U2 pad 8: COL7 -> ROW0
Routing:
- net RESET: track 0.00 -> 133.4 mm
- net BOOT: track 131.8 -> 123.3 mm, vias 0 -> 2
- net ROW2: track 231.5 -> 239.4 mm, vias 0 -> 2
- net GND: track 45.1 -> 52.4 mm
- net ROW0: track 280.6 -> 274.0 mm
- net Net-(D42-A): track 12.2 -> 5.64 mm
- net COL7: track 67.8 -> 61.4 mm
- net ROW3: track 255.9 -> 258.8 mm, vias 0 -> 3
- net +5V: track 38.2 -> 36.8 mm, vias 2 -> 0
- net D-: track 37.8 -> 36.5 mm, vias 2 -> 0
- net Net-(U2-VREF+): track 6.61 -> 7.71 mm
- net COL0: track 219.9 -> 220.8 mm
- net D+: track 37.4 -> 36.5 mm, vias 2 -> 0
